Commit message: fix arm remote

File: src/so101_description/urdf/so101.urdf (robot description, URDF)
Before this commit: robot so101, 8 links, 7 joints
Links:
- removed link link_2
- removed link link_3
- removed link link_4
- removed link link_5
- removed link world
- removed link wrist_roll_follower_so101_v1
- added link gripper_frame_link, mass 1e-9
- added link jaw_tip, mass 1e-9
- added link part_31, mass 0.100006; collision mesh filename=package://so101_description/meshes/part_31.stl; collision mesh filename=package://so101_description/meshes/part_32.stl
- added link part_37, mass 0.103; collision mesh filename=package://so101_description/meshes/part_37.stl; collision mesh filename=package://so101_description/meshes/part_38.stl
- added link part_42, mass 0.104; collision mesh filename=package://so101_description/meshes/part_42.stl; collision mesh filename=package://so101_description/meshes/part_43.stl
- added link part_56, mass 0.087; collision mesh filename=package://so101_description/meshes/part_56.stl; collision mesh filename=package://so101_description/meshes/part_57.stl
- added link part_63, mass 0.079; collision mesh filename=package://so101_description/meshes/part_63.stl; collision mesh filename=package://so101_description/meshes/part_64.stl
- link base_link: mass 0.234577 -> 0.147; geometry collision mesh filename=package://so101_description/meshes/base_arm.stl; collision mesh filename=package://so101_description/meshes/base_arm_servo_cap.stl
- link moving_jaw_so101_v1: mass 0.007332 -> 0.012; geometry collision mesh filename=package://so101_description/meshes/moving_jaw_so101_v1.stl; visual mesh filename=package://so101_description/meshes/moving_jaw_so101_v1.stl
Joints:
- removed joint world_to_base
- added joint gripper_frame_link_frame: type fixed, parent part_56, child gripper_frame_link, origin xyz=-9.3491e-08 -0 -0.114718 rpy=-1.5708 -0 -1e-12, axis 0 0 0
- added joint jaw_tip_frame: type fixed, parent moving_jaw_so101_v1, child jaw_tip, origin xyz=-0.0857177 0.0121501 0.0298826 rpy=-3.14159 -1.57079 1.5708, axis 0 0 0
- joint gripper_joint: axis 0 0 -1 -> 0 0 1; limit lower=-0.451427 upper=0.59577 effort=2.5 velocity=3.0 -> lower=-0 upper=1.5708 effort=2.94 velocity=10; origin xyz=0.019722 -0.026609 0.004746 rpy=0 -1.1612 0 -> xyz=-0.0298825 0.01215 -0.029 rpy=3.14159 -1.5708 0; parent wrist_roll_follower_so101_v1 -> part_56
- joint joint_1: axis 0 1 0 -> 0 0 1; child link_2 -> part_31; limit lower=-3.14159 upper=0.90101 effort=2.5 velocity=3.0 -> lower=-1.5708 upper=1.5708 effort=2.94 velocity=10; origin xyz=0 0.031 0.05955 rpy=0 0 0 -> xyz=-0 -0.05945 0.0303 rpy=-0 0 0
- joint joint_2: axis -1 0 0 -> 0 0 1; child link_3 -> part_37; limit lower=-1.20475 upper=1.93684 effort=2.5 velocity=3.0 -> lower=-1.5708 upper=1.5708 effort=2.94 velocity=10; origin xyz=0.042226 0.11745 -0.012719 rpy=0 1.05471 0 -> xyz=0.0305 -0.03045 0.11355 rpy=0 -1.5708 0; parent link_2 -> part_31
- joint joint_3: axis -1 0 0 -> 0 0 1; child link_4 -> part_42; limit lower=-1.55826 upper=1.23427 effort=2.5 velocity=3.0 -> lower=-1.5708 upper=1.5708 effort=2.94 velocity=10; origin xyz=0 0.106979 0.078865 rpy=0.366045 0 0 -> xyz=0.12647 -0.02745 -0 rpy=-0 0 -0; parent link_3 -> part_37
- joint joint_4: axis -1 0 0 -> 0 0 1; child link_5 -> part_63; limit lower=-0.210268 upper=2.58226 effort=2.5 velocity=3.0 -> lower=-1.5708 upper=1.5708 effort=2.94 velocity=10; origin xyz=0 0.017637 0.139228 rpy=-0.161994 0 0 -> xyz=-0.0025 -0.13015 -0 rpy=0 -0 0; parent link_4 -> part_42
- joint joint_5: axis 0 1 0 -> 0 0 1; child wrist_roll_follower_so101_v1 -> part_56; limit lower=-0.79539 upper=0.78539 effort=2.5 velocity=3.0 -> lower=-6.28319 upper=0 effort=2.94 velocity=10; origin xyz=-0.03205 -0.072077 0.015383 rpy=-0.210268 0 0 -> xyz=-1.35393e-06 -0.0749445 0.0304 rpy=-1.5708 1.5708 0; parent link_5 -> part_63
